File: eagle nodemcu/nodemcu1.sch (EAGLE design)
At the start: 39 parts, among them IC1 MCP23008/P, U1 DS3232MZ+, X1 332-28

Commit message: Add files via upload
Parts:
- removed H3: MOUNT-PAD-ROUND2.8, holes:MOUNT-PAD-ROUND2.8
- added C4: 1.0uF, SparkFun-Capacitors:1.0UF-1206-50V-10%
Connections:
- new net N$1: D2.A, R3.2, R6.1, S1.P
- new net N$2: U$1.3V
- new net N$9: U$1.3V@1
- net 3.3V: now also C4.1; no longer U$1.3V, U$1.3V@1
- net BUTTON: no longer D2.A, R3.2, R6.1, S1.P
- net GND: now also C4.2
Other:
- moved on the sheet: C7
Changed lines of the file:
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@@
 </class>
 <class number="1" name="signal" width="0.254" drill="0.3048">
-<clearance class="1" value="0.254"/>
+<clearance class="1" value="0.3048"/>
 </class>
 <class number="2" name="power" width="0.508" drill="0.6096">
-<clearance class="2" value="0.254"/>
+<clearance class="2" value="0.3048"/>
 </class>
 </classes>
@@
 <part name="H1" library="holes" library_urn="urn:adsk.eagle:library:237" deviceset="MOUNT-PAD-ROUND" device="2.8" package3d_urn="urn:adsk.eagle:package:14281/1" value="MOUNT-PAD-ROUND2.8"/>
 <part name="H2" library="holes" library_urn="urn:adsk.eagle:library:237" deviceset="MOUNT-PAD-ROUND" device="2.8" package3d_urn="urn:adsk.eagle:package:14281/1" value="MOUNT-PAD-ROUND2.8"/>
-<part name="H3" library="holes" library_urn="urn:adsk.eagle:library:237" deviceset="MOUNT-PAD-ROUND" device="2.8" package3d_urn="urn:adsk.eagle:package:14281/1" value="MOUNT-PAD-ROUND2.8"/>
 <part name="H4" library="holes" library_urn="urn:adsk.eagle:library:237" deviceset="MOUNT-PAD-ROUND" device="2.8" package3d_urn="urn:adsk.eagle:package:14281/1" value="MOUNT-PAD-ROUND2.8"/>
 <part name="J2" library="SparkFun-Connectors" deviceset="CONN_08" device="&quot;"/>
 <part name="GND16" library="SparkFun-PowerSymbols" deviceset="GND" device=""/>
+<part name="C4" library="SparkFun-Capacitors" library_urn="urn:adsk.eagle:library:510" deviceset="1.0UF" device="-1206-50V-10%" package3d_urn="urn:adsk.eagle:package:37426/1" value="1.0uF"/>
 </parts>
 <sheets>
@@
 <attribute name="VALUE" x="236.22" y="149.606" size="1.778" layer="96" align="top-center"/>
 </instance>
-<instance part="C7" gate="G$1" x="210.82" y="33.02" smashed="yes" rot="R180">
-<attribute name="NAME" x="209.296" y="30.099" size="1.778" layer="95" font="vector" rot="R180"/>
-<attribute name="VALUE" x="209.296" y="35.179" size="1.778" layer="96" font="vector" rot="R180"/>
+<instance part="C7" gate="G$1" x="208.28" y="33.02" smashed="yes" rot="R180">
+<attribute name="NAME" x="206.756" y="30.099" size="1.778" layer="95" font="vector" rot="R180"/>
+<attribute name="VALUE" x="206.756" y="35.179" size="1.778" layer="96" font="vector" rot="R180"/>
 </instance>
 <instance part="R7" gate="G$1" x="40.64" y="81.28" smashed="yes" rot="R90">
@@
 <attribute name="VALUE" x="73.914" y="195.6562" size="1.778" layer="96"/>
 </instance>
-<instance part="H3" gate="G$1" x="106.68" y="198.12" smashed="yes">
-<attribute name="NAME" x="109.474" y="198.7042" size="1.778" layer="95"/>
-<attribute name="VALUE" x="109.474" y="195.6562" size="1.778" layer="96"/>
-</instance>
 <instance part="H4" gate="G$1" x="142.24" y="198.12" smashed="yes">
 <attribute name="NAME" x="145.034" y="198.7042" size="1.778" layer="95"/>
@@
 <instance part="GND16" gate="1" x="33.02" y="111.76" smashed="yes">
 <attribute name="VALUE" x="33.02" y="111.506" size="1.778" layer="96" align="top-center"/>
+</instance>
+<instance part="C4" gate="G$1" x="213.36" y="35.56" smashed="yes">
+<attribute name="NAME" x="214.884" y="38.481" size="1.778" layer="95" font="vector"/>
+<attribute name="VALUE" x="214.884" y="33.401" size="1.778" layer="96" font="vector"/>
 </instance>
 </instances>
@@
 <pinref part="C7" gate="G$1" pin="1"/>
 <wire x1="220.98" y1="27.94" x2="220.98" y2="25.4" width="0.1524" layer="91"/>
-<wire x1="210.82" y1="27.94" x2="220.98" y2="27.94" width="0.1524" layer="91"/>
 <junction x="220.98" y="27.94"/>
+<wire x1="208.28" y1="27.94" x2="213.36" y2="27.94" width="0.1524" layer="91"/>
+<pinref part="C4" gate="G$1" pin="2"/>
+<wire x1="213.36" y1="27.94" x2="220.98" y2="27.94" width="0.1524" layer="91"/>
+<wire x1="213.36" y1="33.02" x2="213.36" y2="27.94" width="0.1524" layer="91"/>
+<junction x="213.36" y="27.94"/>
 </segment>
 <segment>
@@
 <net name="3.3V" class="2">
 <segment>
-<pinref part="U$1" gate="G$1" pin="3V"/>
-<wire x1="116.84" y1="93.98" x2="114.3" y2="93.98" width="0.1524" layer="91"/>
-<label x="114.3" y="93.98" size="0.6096" layer="95" rot="R180" xref="yes"/>
-</segment>
-<segment>
-<pinref part="U$1" gate="G$1" pin="3V@1"/>
-<wire x1="157.48" y1="83.82" x2="160.02" y2="83.82" width="0.1524" layer="91"/>
-<label x="160.02" y="83.82" size="0.6096" layer="95" xref="yes"/>
-</segment>
-<segment>
 <pinref part="R6" gate="G$1" pin="2"/>
 <wire x1="-30.48" y1="172.72" x2="-30.48" y2="175.26" width="0.1524" layer="91"/>
@@
 <segment>
 <pinref part="SD_HOLDER" gate="G$1" pin="4"/>
-<wire x1="205.74" y1="55.88" x2="210.82" y2="55.88" width="0.1524" layer="91"/>
+<wire x1="205.74" y1="55.88" x2="208.28" y2="55.88" width="0.1524" layer="91"/>
 <label x="215.9" y="55.88" size="0.4064" layer="95" xref="yes"/>
 <pinref part="C7" gate="G$1" pin="2"/>
-<wire x1="210.82" y1="55.88" x2="215.9" y2="55.88" width="0.1524" layer="91"/>
-<wire x1="210.82" y1="35.56" x2="210.82" y2="55.88" width="0.1524" layer="91"/>
-<junction x="210.82" y="55.88"/>
+<wire x1="208.28" y1="55.88" x2="213.36" y2="55.88" width="0.1524" layer="91"/>
+<wire x1="213.36" y1="55.88" x2="215.9" y2="55.88" width="0.1524" layer="91"/>
+<wire x1="208.28" y1="35.56" x2="208.28" y2="55.88" width="0.1524" layer="91"/>
+<junction x="208.28" y="55.88"/>
+<pinref part="C4" gate="G$1" pin="1"/>
+<wire x1="213.36" y1="40.64" x2="213.36" y2="55.88" width="0.1524" layer="91"/>
+<junction x="213.36" y="55.88"/>
 </segment>
 <segment>
@@
 <net name="BUTTON" class="2">
 <segment>
-<pinref part="R6" gate="G$1" pin="1"/>
-<pinref part="D2" gate="G$1" pin="A"/>
-<wire x1="-30.48" y1="160.02" x2="-30.48" y2="162.56" width="0.1524" layer="91"/>
-<wire x1="-25.4" y1="160.02" x2="-30.48" y2="160.02" width="0.1524" layer="91"/>
-<pinref part="S1" gate="G$1" pin="P"/>
-<pinref part="R3" gate="G$1" pin="2"/>
-<wire x1="-30.48" y1="152.4" x2="-30.48" y2="154.94" width="0.1524" layer="91"/>
-<wire x1="-30.48" y1="154.94" x2="-30.48" y2="160.02" width="0.1524" layer="91"/>
-<junction x="-30.48" y="154.94"/>
-<junction x="-30.48" y="160.02"/>
-</segment>
-<segment>
+<wire x1="-17.78" y1="152.4" x2="-15.24" y2="152.4" width="0.1524" layer="91"/>
+<label x="-15.24" y="152.4" size="0.4064" layer="95" xref="yes"/>
+<pinref part="R3" gate="G$1" pin="1"/>
+<wire x1="-20.32" y1="154.94" x2="-17.78" y2="154.94" width="0.1524" layer="91"/>
+<wire x1="-17.78" y1="154.94" x2="-17.78" y2="152.4" width="0.1524" layer="91"/>
 <pinref part="C2" gate="G$1" pin="1"/>
-<wire x1="-17.78" y1="160.02" x2="-17.78" y2="154.94" width="0.1524" layer="91"/>
-<pinref part="R3" gate="G$1" pin="1"/>
-<wire x1="-17.78" y1="154.94" x2="-17.78" y2="152.4" width="0.1524" layer="91"/>
-<wire x1="-17.78" y1="152.4" x2="-17.78" y2="149.86" width="0.1524" layer="91"/>
-<wire x1="-20.32" y1="154.94" x2="-17.78" y2="154.94" width="0.1524" layer="91"/>
-<junction x="-17.78" y="154.94"/>
+<wire x1="-17.78" y1="149.86" x2="-17.78" y2="152.4" width="0.1524" layer="91"/>
+<junction x="-17.78" y="152.4"/>
 <pinref part="D2" gate="G$1" pin="C"/>
 <wire x1="-20.32" y1="160.02" x2="-17.78" y2="160.02" width="0.1524" layer="91"/>
-<wire x1="-17.78" y1="152.4" x2="-15.24" y2="152.4" width="0.1524" layer="91"/>
-<junction x="-17.78" y="152.4"/>
-<label x="-15.24" y="152.4" size="0.4064" layer="95" xref="yes"/>
+<wire x1="-17.78" y1="160.02" x2="-17.78" y2="152.4" width="0.1524" layer="91"/>
 </segment>
 <segment>
@@
 </segment>
 </net>
+<net name="N$1" class="0">
+<segment>
+<pinref part="S1" gate="G$1" pin="P"/>
+<pinref part="R3" gate="G$1" pin="2"/>
+<wire x1="-30.48" y1="152.4" x2="-30.48" y2="154.94" width="0.1524" layer="91"/>
+<wire x1="-30.48" y1="154.94" x2="-30.48" y2="160.02" width="0.1524" layer="91"/>
+<junction x="-30.48" y="154.94"/>
+<pinref part="D2" gate="G$1" pin="A"/>
+<wire x1="-30.48" y1="160.02" x2="-25.4" y2="160.02" width="0.1524" layer="91"/>
+<pinref part="R6" gate="G$1" pin="1"/>
+<wire x1="-30.48" y1="162.56" x2="-30.48" y2="154.94" width="0.1524" layer="91"/>
+</segment>
+</net>
+<net name="N$2" class="0">
+<segment>
+<pinref part="U$1" gate="G$1" pin="3V"/>
+<wire x1="116.84" y1="93.98" x2="116.078" y2="93.98" width="0.1524" layer="91"/>
+</segment>
+</net>
+<net name="N$9" class="0">
+<segment>
+<pinref part="U$1" gate="G$1" pin="3V@1"/>
+<wire x1="157.48" y1="83.82" x2="158.496" y2="83.82" width="0.1524" layer="91"/>
+</segment>
+</net>
