File: eagle nodemcu/nodemcu1_with converter.sch (EAGLE design)
At the start: 39 parts, among them IC1 MCP23008/P, U1 DS3232MZ+, X1 332-28

Commit message: Add files via upload
Parts:
- removed H3: MOUNT-PAD-ROUND2.8, holes:MOUNT-PAD-ROUND2.8
- added C4: 1.0uF, SparkFun-Capacitors:1.0UF-1206-50V-10%
- added D1: 1N4148WS, Diodes:1N4148WS
- added R17: 10.43k, SparkFun-Resistors:0.22OHM-0805-1/4W-1%
- added R18: 750, SparkFun-Resistors:0.22OHM-0805-1/4W-1%
- added T1: BC847, transistor:BC847
Connections:
- new net N$1: D2.A, R3.2, R6.1, S1.P
- new net N$10: D1.C, R17.2, T1.B
- new net N$9: U$1.3V@1
- net 3.3V: now also C4.1, R18.1; no longer U$1.3V@1
- net BUTTON: no longer D2.A, R3.2, R6.1, S1.P
- net ESP_RX: now also R18.2, T1.C
- net GND: now also C4.2, D1.A, T1.E
- net TX_MIDMARK: now also R17.1
Other:
- note added: "MIDMARK M11_NEW"
- note added: "OLD MIDMARKS"
- moved on the sheet: C7
